File: schematics/ARCHIVE/MEASURE_IF-v1.0.1/MEASURE_IF.kicad_pcb (KiCad board)
At the start: 2 copper layers, 45.7 x 65.2 mm, 49 parts, among them J1 SWD_CONN, J2 ARGUS_SPI_LEGACY_CONN, J4 VMOT_IN_5mm, J5 MOT_TERM, J6 MOT_TERM, J7 USB_B_Micro, J8 MOT_TERM, J9 MOT_TERM, SW1 SW_RESET, U1 LD3985M33R_SOT23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

Commit message: Improve board artwork
Parts:
- added J3: ARGUS_SPI_FFC_CONN, Connector_FFC-FPC:Hirose_FH12-10S-0.5SH_1x10-1MP_P0.50mm_Horizontal, F.Cu at (30.5, 142.7)
- moved J2 1.28 mm to (35.6, 141.5), turned to 0 degrees
Routing:
- net GND: track 199.5 -> 182.6 mm
- net VSSA: track 41.2 -> 58.0 mm
- net /SPI_SCK: track 12.3 -> 22.9 mm
- net /SPI_MOSI: track 15.0 -> 23.0 mm
- net /ARGUS_CS: track 11.7 -> 17.5 mm, vias 0 -> 1
- net VCC: track 149.1 -> 153.9 mm, vias 3 -> 5
- net /NRST: track 96.3 -> 93.9 mm
- net /SPI_MISO: track 15.6 -> 18.0 mm
- net /MOTuCONF1: track 58.7 -> 59.4 mm
Other:
- board text removed: "GND"
- board text removed: "SWCLK"
- board text removed: "SWDIO"
- board text removed: "VCC"
